File: headphone_amplifier_board/Headphone_Amp.kicad_pcb (KiCad board)
At the start: 2 copper layers, 150 x 56.4 mm, 144 parts, among them J1 PWR_IN, J2 Headphone_IN, J3 Audio_IN, J4 Conn_01x03, J5 Conn_01x03, T1 SSM3J338R_LF, U1 NE5532, U10 NE5532, U11 NE5532, U12 NE5532, U13 NE5532, U14 NE5532, U15 NE5532, U16 NE5532, U17 NE5532, U18 NE5532, U19 LM317_TO-252, U2 NE5532, U3 NE5532, U4 NE5532, U5 NE5532, U6 NE5532, U7 NE5532, U8 NE5532, U9 NE5532

Commit message: Bug Fix
Parts:
- moved R3 58.2 mm to (158.8, 55.5), turned to -90 degrees
- moved R4 51.1 mm to (155.2, 55.5)
- moved C19 16.7 mm to (139.0, 77.0)
- moved C14 15.5 mm to (144.9, 62.8)
- moved U4 15.2 mm to (138.5, 64.5)
- moved C18 6.79 mm to (157.2, 65.0)
- moved R18 6.79 mm to (157.0, 69.0)
- moved R17 2.85 mm to (162.5, 55.5)
- moved R19 2.06 mm to (148.5, 56.5)
- moved C17 0.89 mm to (162.5, 47.5)
- moved C16 0.85 mm to (158.8, 47.5)
Routing:
- net Net-(D4-A1): track 0.00 -> 15.3 mm
- net Net-(D5-A1): track 0.00 -> 15.2 mm
- net AUDIO_IN_RIGHT: track 0.00 -> 5.96 mm
- net AUDIO_IN_LEFT: track 0.00 -> 5.96 mm
- net GND: track 33.3 -> 38.4 mm, vias 17 -> 19
- net +15V: track 89.0 -> 92.0 mm

Commit message: updated routing
Parts:
- added G***: LOGO, LOGO, F.Cu at (169.0, 35.2)
- moved R55 150.8 mm to (179.2, 88.9)
- moved R65 145.8 mm to (179.3, 96.5)
- moved C42 141.9 mm to (179.2, 85.5)
- moved R54 139.9 mm to (167.0, 86.3), turned to -90 degrees
- moved R47 139.6 mm to (161.7, 89.1)
- moved R45 139.6 mm to (144.5, 89.3)
- moved C47 135.3 mm to (179.3, 93.1)
- moved R64 135.0 mm to (167.1, 94.1), turned to -90 degrees
- moved H4 134.1 mm to (75.9, 108.8)
- moved C37 133.2 mm to (161.8, 85.7)
- moved U14 131.0 mm to (172.7, 87.2)
- moved R44 129.7 mm to (131.5, 86.6), turned to -90 degrees
- moved C31 129.2 mm to (106.3, 66.8)
- moved R46 129.1 mm to (149.6, 86.6), turned to -90 degrees
- moved R63 127.7 mm to (161.8, 96.7)
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Routing:
- net PREAMP_OUT_RIGHT: track 0.00 -> 130.5 mm
- net PREAMP_OUT_LEFT: track 0.00 -> 130.0 mm
- net DRIVER_OUT_LEFT: track 0.00 -> 123.4 mm
- net GND: track 38.4 -> 158.4 mm, vias 19 -> 81
- net DRIVER_OUT_RIGHT: track 0.00 -> 116.0 mm
- net VBIAS_LEFT: track 7.83 -> 123.2 mm, vias 0 -> 6
- net VBIAS_RIGHT: track 8.09 -> 97.7 mm, vias 0 -> 6
- net Net-(U3B-+): track 0.00 -> 50.0 mm
- net Net-(U6A--): track 0.00 -> 47.6 mm
- net INP_BUF_OUT_RIGHT: track 0.00 -> 45.2 mm
- net Net-(U5A--): track 0.00 -> 44.4 mm
- net Net-(U4B-+): track 0.00 -> 41.6 mm
- net INP_BUF_OUT_LEFT: track 0.00 -> 39.7 mm
- net Net-(J5-Pin_3): track 0.00 -> 38.9 mm
- net +15V: track 92.0 -> 126.3 mm, vias 0 -> 21
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- added copper zone on In2.Cu, net +15V
- added copper zone on B.Cu, net GND
- added copper zone on In1.Cu, net GND
Other:
- board size 150 x 56.4 mm -> 111.7 x 81.2 mm
- copper layers 2 -> 4
- board text added: "BIAS LEFT"
- board text added: "BIAS RIGHT"
- board text added: "GiugSystems"
- board text added: "HEADPHONE_AMP"
- board text added: "JLCJLCJLCJLC"
- board text added: "L"
- board text added: "LEFT CH"
- board text added: "PSU SECTION"
- board text added: "R"
- board text added: "RIGHT CH"
- board text added: "Rev 1.0"
